Commit message: camera set

File: my_robo_test/my_robo_d/urdf/ball1.xacro (robot description, xacro)
@@ -3,4 +3,5 @@
   <xacro:include filename="$(find test_gazebo_camera)/urdf/ball1.gazebo"/>
   <xacro:include filename="$(find test_gazebo_camera)/urdf/materials.xacro"/>
+  <xacro:property name="x" value="1.0"/>
   <link name="world"/>
   <joint name="fix" type="fixed">
@@ -11,5 +12,5 @@
   <link name="link1">
     <collision>
-      <origin xyz = "1.5 0 1.5" rpy="0 0 0"/>
+      <origin xyz = "${x} 0 1.5" rpy="0 0 0"/>
       <geometry>
         <sphere radius="0.1"/>
@@ -17,5 +18,5 @@
     </collision>
     <visual>
-      <origin xyz = "1.5 0 1.5" rpy="0 0 0"/>
+      <origin xyz = "${x} 0 1.5" rpy="0 0 0"/>
       <geometry>
         <sphere radius="0.1"/>
@@ -25,5 +26,5 @@
     <inertial>
       <mass value = "0.1"/>
-      <origin xyz = "1.5 0 1.5" rpy="0 0 0"/>
+      <origin xyz = "${x} 0 1.5" rpy="0 0 0"/>
       <inertia ixx="0.0001" ixy = "0" ixz = "0" iyy= "0.0001" iyz="0" izz="0.0001"/>
     </inertial>

File: my_robo_test/my_robo_d/urdf/box1.xacro (robot description, xacro)
@@ -3,4 +3,5 @@
   <xacro:include filename="$(find test_gazebo_camera)/urdf/box1.gazebo"/>
   <xacro:include filename="$(find test_gazebo_camera)/urdf/materials.xacro"/>
+  <xacro:property name="x" value="1.0"/>
   <link name="world"/>
   <joint name="fix" type="fixed">
@@ -11,5 +12,5 @@
   <link name="link1">
     <collision>
-      <origin xyz = "1.5 0 0.7" rpy="0 0 0"/>
+      <origin xyz = "${x} 0 0.7" rpy="0 0 0"/>
       <geometry>
         <box size = "0.4 0.4 1.4" rpy="0 0 0"/>
@@ -17,5 +18,5 @@
     </collision>
     <visual>
-      <origin xyz = "1.5 0 0.7" rpy="0 0 0"/>
+      <origin xyz = "${x} 0 0.7" rpy="0 0 0"/>
       <geometry>
         <box size = "0.4 0.4 1.4" rpy="0 0 0"/>
@@ -25,5 +26,5 @@
     <inertial>
       <mass value = "0.001"/>
-      <origin xyz = "1.5 0 0.7" rpy="0 0 0"/>
+      <origin xyz = "${x} 0 0.7" rpy="0 0 0"/>
       <inertia ixx="0.0001" ixy = "0" ixz = "0" iyy= "0.0001" iyz="0" izz="0.0001"/>
     </inertial>

File: my_robo_test/my_robo_d/urdf/my_robo.xacro (robot description, xacro)
@@ -11,5 +11,5 @@
   <xacro:property name="width3" value="0.4"/>
   <xacro:property name="width4" value="0.4"/>
-  <xacro:property name="width5" value="0.2"/>
+  <xacro:property name="width5" value="0.01"/>
   <xacro:property name="width6" value="0.025"/>
   <xacro:property name="size_cam" value="0.03"/>

Commit message: gripper

File: my_robo_test/my_robo_d/urdf/ball1.xacro (robot description, xacro)
@@ -3,6 +3,9 @@
   <xacro:include filename="$(find test_gazebo_camera)/urdf/ball1.gazebo"/>
   <xacro:include filename="$(find test_gazebo_camera)/urdf/materials.xacro"/>
-  <xacro:property name="x" value="1.0"/>
-  <link name="world"/>
+  <xacro:property name="x" value="0.3"/>
+  <xacro:property name="y" value="0.0"/>
+  <xacro:property name="r" value="0.02"/>
+  <xacro:property name="z" value="${r}"/>
+  <!--<link name="world"/>
   <joint name="fix" type="fixed">
     <origin xyz = "0 0 0" rpy="0 0 0"/>
@@ -10,21 +13,22 @@
     <child link = "link1"/>
   </joint>
+-->
   <link name="link1">
     <collision>
-      <origin xyz = "${x} 0 1.5" rpy="0 0 0"/>
+      <origin xyz = "${x} ${y} ${z}" rpy="0 0 0"/>
       <geometry>
-        <sphere radius="0.1"/>
+        <sphere radius="${r}"/>
       </geometry>
     </collision>
     <visual>
-      <origin xyz = "${x} 0 1.5" rpy="0 0 0"/>
+      <origin xyz = "${x} ${y} ${z}" rpy="0 0 0"/>
       <geometry>
-        <sphere radius="0.1"/>
+        <sphere radius="${r}"/>
       </geometry>
       <material name="red"/>
     </visual>
     <inertial>
-      <mass value = "0.1"/>
-      <origin xyz = "${x} 0 1.5" rpy="0 0 0"/>
+      <mass value = "0.005"/>
+      <origin xyz = "${x} ${y} ${z}" rpy="0 0 0"/>
       <inertia ixx="0.0001" ixy = "0" ixz = "0" iyy= "0.0001" iyz="0" izz="0.0001"/>
     </inertial>

File: my_robo_test/my_robo_d/urdf/my_robo.xacro (robot description, xacro)
@@ -2,19 +2,27 @@
 <robot name="my_robo" xmlns:xacro="http://www.ros.org/wiki/xacro">
   <xacro:property name="PI" value="3.1415926535"/>
-  <xacro:property name="mass1" value="3.0"/>
-  <xacro:property name="mass2" value="3.0"/>
-  <xacro:property name="mass3" value="3.0"/>
-  <xacro:property name="mass4" value="3.0"/>
-  <xacro:property name="mass5" value="3.0"/>
+  <xacro:property name="mass1" value="0.05"/>
+  <xacro:property name="mass2" value="0.05"/>
+  <xacro:property name="mass3" value="0.05"/>
+  <xacro:property name="mass4" value="0.02"/>
+  <xacro:property name="mass5" value="0.02"/>
   <xacro:property name="width1" value="0.1"/>
   <xacro:property name="width2" value="0.1"/>
-  <xacro:property name="width3" value="0.4"/>
-  <xacro:property name="width4" value="0.4"/>
+  <xacro:property name="width3" value="0.2"/>
+  <xacro:property name="width4" value="0.2"/>
   <xacro:property name="width5" value="0.01"/>
-  <xacro:property name="width6" value="0.025"/>
-  <xacro:property name="size_cam" value="0.03"/>
+  <xacro:property name="width6" value="0.01"/>
+  <xacro:property name="width7" value="0.01"/>
+  <xacro:property name="ha" value="0.08"/>
+  <xacro:property name="size_cam" value="0.01"/>
   <xacro:property name="offset_cam" value="0.03"/>
+  <xacro:property name="low" value="-1.57"/>
+  <xacro:property name="up" value="1.57"/>
+  <xacro:property name="eff" value="10.0"/>
+  <xacro:property name="vel" value="5.0"/>
   <xacro:property name="sizeX" value="0.05"/>
   <xacro:property name="sizeY" value="0.05"/>
+  <xacro:property name="sizeXg" value="0.05"/>
+  <xacro:property name="sizeYg" value="0.05"/>
   <xacro:property name="offsetX" value="0.01"/>
   <xacro:property name="offsetY" value="0.05"/>
@@ -23,5 +31,5 @@
   <link name="world"/>
   <joint name="fixed" type="fixed">
-    <origin xyz="0 0 1.7" rpy="0 0 0"/>
+    <origin xyz="0 0 0.4" rpy="0 0 0"/>
     <parent link="world"/>
     <child link="link1"/>
@@ -31,5 +39,5 @@
       <origin xyz="${width1/2} 0 0" rpy="0 0 0"/>
       <geometry>
-        <box size="${width1} ${sizeX} ${sizeY}"/>
+        <box size="${width1/2} ${sizeX/2} ${sizeY/2}"/>
       </geometry>
     </collision>
@@ -50,5 +58,5 @@
     </inertial>
   </link>
-  <joint name="joint1" type="continuous">
+  <joint name="joint1" type="revolute">
     <origin xyz="${width1+offsetX} 0 0" rpy="0 0 0"/>
     <parent link="link1"/>
@@ -56,4 +64,5 @@
     <axis xyz ="1 0 0"/>
     <dynamics damping="0.7"/>
+    <limit lower = "${low}" upper = "${up}" effort="${eff}" velocity="${vel}"/>
   </joint>
   <link name="link2">
@@ -80,5 +89,5 @@
     </inertial>
   </link>
-  <joint name="joint2" type="continuous">
+  <joint name="joint2" type="revolute">
     <origin xyz="${width2-offsetY} ${offsetY} 0" rpy="0 0 0"/>
     <parent link="link2"/>
@@ -86,4 +95,5 @@
     <axis xyz ="0 1 0"/>
     <dynamics damping="0.7"/>
+    <limit lower = "${low}" upper = "${up}" effort="${eff}" velocity="${vel}"/>
   </joint>
   <link name="link3">
@@ -110,5 +120,5 @@
     </inertial>
   </link>
-  <joint name="joint3" type="continuous">
+  <joint name="joint3" type="revolute">
     <origin xyz="${width3-offsetY} ${-offsetY} 0" rpy="0 0 0"/>
     <parent link="link3"/>
@@ -116,4 +126,5 @@
     <axis xyz ="0 1 0"/>
     <dynamics damping="0.7"/>
+    <limit lower = "${low}" upper = "${up}" effort="${eff}" velocity="${vel}"/>
   </joint>
   <link name="link4">
@@ -140,9 +151,10 @@
     </inertial>
   </link>
-  <joint name="joint4" type="continuous">
+  <joint name="joint4" type="revolute">
     <origin xyz="${width4+offsetX} 0 0" rpy="0 0 0"/>
     <parent link="link4"/>
     <child link="link5"/>
     <axis xyz ="1 0 0"/>
+    <limit lower = "${low}" upper = "${up}" effort="${eff}" velocity="${vel}"/>
     <dynamics damping="0.7"/>
   </joint>
@@ -170,25 +182,235 @@
     </inertial>
   </link>
-  <joint name="joint5" type="fixed">
-    <origin xyz="${width5+offsetX} 0 0" rpy="0 0 0"/>
+<!--up_grip-->
+  <joint name="joint5" type="revolute">
+    <origin xyz="${width5} 0 0" rpy="0 0 0"/>
     <parent link="link5"/>
     <child link="link6"/>
+    <limit lower = "${low}" upper = "${up}" effort="${eff}" velocity="${vel}"/>
+    <dynamics damping="0.7"/>
+    <axis xyz="0 1 0"/>
   </joint>
   <link name="link6">
     <collision>
-      <origin xyz="${width6/2} 0 0" rpy="0 0 0"/>
-      <geometry>
-        <box size="${width6/2} ${sizeX/2} ${sizeY/2}"/>
-      </geometry>
-    </collision>
-    <visual>
-      <origin xyz="${width6/2} 0 0" rpy="0 0 0"/>
-      <geometry>
-        <box size="${width6/2} ${sizeX/2} ${sizeY/2}"/>
-      </geometry>
-      <material name="black"/>
-    </visual>
-    <inertial>
-      <origin xyz="${width6/2} 0 0" rpy="0 0 0"/>
+      <origin xyz="${width6} 0 0.03" rpy="0 0 0"/>
+      <geometry>
+        <box size="${width6} ${sizeXg/2} ${sizeYg/2}"/>
+      </geometry>
+    </collision>
+    <visual>
+      <origin xyz="${width6} 0 0.03" rpy="0 0 0"/>
+      <geometry>
+        <box size="${width6} ${sizeXg} ${sizeYg}"/>
+      </geometry>
+      <material name="black"/>
+    </visual>
+    <inertial>
+      <origin xyz="${width6/2} 0 0.03" rpy="0 0 0"/>
+      <mass value="${mass5}"/>
+      <inertia
+        ixx="${mass5 / 12.0 * (width6*width6 + sizeY*sizeY)}" ixy="0.0" ixz="0.0"
+        iyy="${mass5 / 12.0 * (sizeY*sizeY + sizeX * sizeX)}" iyz="0.0"
+        izz="${mass5 / 12.0 * (sizeX * sizeX + width6 * width6)}" />
+    </inertial>
+  </link>
+<!-- up grip2-->
+  <joint name="joint7" type="fixed">
+    <origin xyz="${width5} 0 0" rpy="0 0 0"/>
+    <parent link="link6"/>
+    <child link="link8"/>
+  </joint>
+  <link name="link8">
+    <collision>
+      <origin xyz="0.035 0 0.075" rpy="0 -0.75 0"/>
+      <geometry>
+        <box size="0.06 ${sizeXg} 0.01"/>
+      </geometry>
+    </collision>
+    <visual>
+      <origin xyz="0.03 0 0.075" rpy="0 -0.75 0"/>
+      <geometry>
+        <box size="0.06 ${sizeXg} 0.01"/>
+      </geometry>
+      <material name="black"/>
+    </visual>
+    <inertial>
+      <origin xyz="${width6/2} 0 0.075" rpy="0 -0.75 0"/>
+      <mass value="${mass5}"/>
+      <inertia
+        ixx="${mass5 / 12.0 * (width6*width6 + sizeY*sizeY)}" ixy="0.0" ixz="0.0"
+        iyy="${mass5 / 12.0 * (sizeY*sizeY + sizeX * sizeX)}" iyz="0.0"
+        izz="${mass5 / 12.0 * (sizeX * sizeX + width6 * width6)}" />
+    </inertial>
+  </link>
+<!-- up grip3-->
+  <joint name="joint9" type="fixed">
+    <origin xyz="0 0 0" rpy="0 0 0"/>
+    <parent link="link8"/>
+    <child link="link10"/>
+  </joint>
+  <link name="link10">
+    <collision>
+      <origin xyz="0.035 0.03 0.065" rpy="0 0.75 0"/>
+      <geometry>
+        <box size="0.01 0.01 ${ha/2}"/>
+      </geometry>
+    </collision>
+    <visual>
+      <origin xyz="0.03 0.03 0.065" rpy="0 0.75 0"/>
+      <geometry>
+        <box size="0.01 0.01 ${ha}"/>
+      </geometry>
+      <material name="black"/>
+    </visual>
+    <inertial>
+      <origin xyz="0.03 0.03 0.065" rpy="0 0.75 0"/>
+      <mass value="${mass5}"/>
+      <inertia
+        ixx="${mass5 / 12.0 * (width6*width6 + sizeY*sizeY)}" ixy="0.0" ixz="0.0"
+        iyy="${mass5 / 12.0 * (sizeY*sizeY + sizeX * sizeX)}" iyz="0.0"
+        izz="${mass5 / 12.0 * (sizeX * sizeX + width6 * width6)}" />
+    </inertial>
+  </link>
+<!-- up grip4-->
+  <joint name="joint10" type="fixed">
+    <origin xyz="0 0 0" rpy="0 0 0"/>
+    <parent link="link8"/>
+    <child link="link11"/>
+  </joint>
+  <link name="link11">
+    <collision>
+      <origin xyz="0.035 -0.03 0.065" rpy="0 0.75 0"/>
+      <geometry>
+        <box size="0.01 0.01 ${ha/2}"/>
+      </geometry>
+    </collision>
+    <visual>
+      <origin xyz="0.03 -0.03 0.065" rpy="0 0.75 0"/>
+      <geometry>
+        <box size="0.01 0.01 ${ha}"/>
+      </geometry>
+      <material name="black"/>
+    </visual>
+    <inertial>
+      <origin xyz="0.03 -0.03 0.065" rpy="0 0.75 0"/>
+      <mass value="${mass5}"/>
+      <inertia
+        ixx="${mass5 / 12.0 * (width6*width6 + sizeY*sizeY)}" ixy="0.0" ixz="0.0"
+        iyy="${mass5 / 12.0 * (sizeY*sizeY + sizeX * sizeX)}" iyz="0.0"
+        izz="${mass5 / 12.0 * (sizeX * sizeX + width6 * width6)}" />
+    </inertial>
+  </link>
+<!--down grip-->
+  <joint name="joint6" type="revolute">
+    <origin xyz="${width5} 0 0" rpy="0 0 0"/>
+    <parent link="link5"/>
+    <child link="link7"/>
+    <limit lower = "${low}" upper = "${up}" effort="${eff}" velocity="${vel}"/>
+    <dynamics damping="0.7"/>
+    <axis xyz="0 -1 0"/>
+  </joint>
+  <link name="link7">
+    <collision>
+      <origin xyz="${width6} 0 -0.03" rpy="0 0 0"/>
+      <geometry>
+        <box size="${width6} ${sizeXg/2} ${sizeYg/2}"/>
+      </geometry>
+    </collision>
+    <visual>
+      <origin xyz="${width6} 0 -0.03" rpy="0 0 0"/>
+      <geometry>
+        <box size="${width6} ${sizeXg} ${sizeYg}"/>
+      </geometry>
+      <material name="black"/>
+    </visual>
+    <inertial>
+      <origin xyz="${width6/2} 0 -0.03" rpy="0 0 0"/>
+      <mass value="${mass5}"/>
+      <inertia
+        ixx="${mass5 / 12.0 * (width6*width6 + sizeY*sizeY)}" ixy="0.0" ixz="0.0"
+        iyy="${mass5 / 12.0 * (sizeY*sizeY + sizeX * sizeX)}" iyz="0.0"
+        izz="${mass5 / 12.0 * (sizeX * sizeX + width6 * width6)}" />
+    </inertial>
+  </link>
+<!--down grip2-->
+  <joint name="joint8" type="fixed">
+    <origin xyz="${width5} 0 0" rpy="0 0 0"/>
+    <parent link="link7"/>
+    <child link="link9"/>
+  </joint>
+  <link name="link9">
+    <collision>
+      <origin xyz="0.035 0 -0.075" rpy="0 0.75 0"/>
+      <geometry>
+        <box size="0.06 ${sizeXg} 0.01"/>
+      </geometry>
+    </collision>
+    <visual>
+      <origin xyz="0.03 0 -0.075" rpy="0 0.75 0"/>
+      <geometry>
+        <box size="0.06 ${sizeXg} 0.01"/>
+      </geometry>
+      <material name="black"/>
+    </visual>
+    <inertial>
+      <origin xyz="${width6/2} 0 -0.075" rpy="0 0.75 0"/>
+      <mass value="${mass5}"/>
+      <inertia
+        ixx="${mass5 / 12.0 * (width6*width6 + sizeY*sizeY)}" ixy="0.0" ixz="0.0"
+        iyy="${mass5 / 12.0 * (sizeY*sizeY + sizeX * sizeX)}" iyz="0.0"
+        izz="${mass5 / 12.0 * (sizeX * sizeX + width6 * width6)}" />
+    </inertial>
+  </link>
+<!-- down grip3-->
+  <joint name="joint11" type="fixed">
+    <origin xyz="0 0 0" rpy="0 0 0"/>
+    <parent link="link9"/>
+    <child link="link12"/>
+  </joint>
+  <link name="link12">
+    <collision>
+      <origin xyz="0.035 0.03 -0.065" rpy="0 -0.75 0"/>
+      <geometry>
+        <box size="0.01 0.01 ${ha/2}"/>
+      </geometry>
+    </collision>
+    <visual>
+      <origin xyz="0.03 0.03 -0.065" rpy="0 -0.75 0"/>
+      <geometry>
+        <box size="0.01 0.01 ${ha}"/>
+      </geometry>
+      <material name="black"/>
+    </visual>
+    <inertial>
+      <origin xyz="0.03 0.03 -0.065" rpy="0 -0.75 0"/>
+      <mass value="${mass5}"/>
+      <inertia
+        ixx="${mass5 / 12.0 * (width6*width6 + sizeY*sizeY)}" ixy="0.0" ixz="0.0"
+        iyy="${mass5 / 12.0 * (sizeY*sizeY + sizeX * sizeX)}" iyz="0.0"
+        izz="${mass5 / 12.0 * (sizeX * sizeX + width6 * width6)}" />
+    </inertial>
+  </link>
+<!-- down grip4-->
+  <joint name="joint12" type="fixed">
+    <origin xyz="0 0 0" rpy="0 0 0"/>
+    <parent link="link9"/>
+    <child link="link13"/>
+  </joint>
+  <link name="link13">
+    <collision>
+      <origin xyz="0.03 -0.03 -0.065" rpy="0 -0.75 0"/>
+      <geometry>
+        <box size="0.01 0.01 ${ha/2}"/>
+      </geometry>
+    </collision>
+    <visual>
+      <origin xyz="0.03 -0.03 -0.065" rpy="0 -0.75 0"/>
+      <geometry>
+        <box size="0.01 0.01 ${ha}"/>
+      </geometry>
+      <material name="black"/>
+    </visual>
+    <inertial>
+      <origin xyz="0.03 -0.03 -0.065" rpy="0 -0.75 0"/>
       <mass value="${mass5}"/>
       <inertia
@@ -334,3 +556,23 @@
     </actuator>
   </transmission>
+  <transmission name="tran5">
+    <type>transmission_interface/SimpleTransmission</type>
+    <joint name="joint5">
+      <hardwareInterface>hardware_interface/VelocityJointInterface</hardwareInterface>
+    </joint>
+    <actuator name="motor5">
+      <hardwareInterface>hardware_interface/VelocityJointInterface</hardwareInterface>
+      <mechanicalReduction>1</mechanicalReduction>
+    </actuator>
+  </transmission>
+  <transmission name="tran6">
+    <type>transmission_interface/SimpleTransmission</type>
+    <joint name="joint6">
+      <hardwareInterface>hardware_interface/VelocityJointInterface</hardwareInterface>
+    </joint>
+    <actuator name="motor6">
+      <hardwareInterface>hardware_interface/VelocityJointInterface</hardwareInterface>
+      <mechanicalReduction>1</mechanicalReduction>
+    </actuator>
+  </transmission>
 </robot>
